File: TPS56A37RPAR.kicad_sch (KiCad schematic)
At the start: 26 parts, among them U1 TPS56A37RPAR, U2 LM5165YQDRCTQ1

Commit message: Added final missing footprints, ready to set drc
Parts:
- BT1: footprint (none) -> Connector_BarrelJack:BarrelJack_CUI_PJ-063AH_Horizontal
- C9: value 10u -> 22u
- L1: footprint (none) -> Library:L_Wurth_WE-HCI-1890
- L2: footprint (none) -> Library:IND_LPS4018-473MRC
Other:
- note added: "LM5165Y-Q1 24V -> 3.3V PFM MODE (ref: TI SNVSAJ3C, Design 2) Vin(nom)=24V Vin(op)=24-28V Vin(max)=32V (rail limit, TPS56A37 abs max) Vout=3.3V (fixed, Y version) Iout(target)=50mA Iout(max)=60mA MODE: RT tied to GND -> PFM (light-load efficiency) R_ILIM = 56.2k (1%) -> Ipk = 120mA PFM: Iout(max) = Ipk/2 = 60mA (design target 50mA) L_F = 47uH, Isat >= 0.5A (Coilcraft LPS4018-473MRC) Eq.19: Fsw = (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"
- note removed: "LM5165Y-Q1 24V -> 3.3V PFM MODE (ref: TI SNVSAJ3C, Design 2) Vin(nom)=24V Vin(max)=45V (TVS clamp) Vout=3.3V Iout(max)=50mA MODE: RT tied to GND -> PFM (light-load efficiency, Iout max 100mA) R_ILIM = 56.2k (1%) -> Ipk = 120mA PFM: Iout(max) = Ipk/2 = 60mA (design target 50mA) L_F = 47uH, Isat >= 0.5A (Coilcraft LPS4018-473MRC) Eq.19: Fsw = (Vout/(L*Ipk)) * (1 - Vout/Vin) Ipk = 120mA * 1.1 = 132m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"
Changed lines of the file:
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@@
 		)
 	)
-	(text "LM5165Y-Q1  24V -> 3.3V  PFM MODE  (ref: TI SNVSAJ3C, Design 2)\nVin(nom)=24V  Vin(max)=45V (TVS clamp)  Vout=3.3V  Iout(max)=50mA\n\nMODE: RT tied to GND -> PFM (light-load efficiency, Iout max 100mA)\n\nR_ILIM = 56.2k (1%) -> Ipk = 120mA\n  PFM: Iout(max) = Ipk/2 = 60mA  (design target 50mA)\n\nL_F = 47uH, Isat >= 0.5A  (Coilcraft LPS4018-473MRC)\n  Eq.19: Fsw = (Vout/(L*Ipk)) * (1 - Vout/Vin)\n         Ipk = 120mA * 1.1 = 132mA (comparator delay margin)\n         Fsw @24V = (3.3/(47u*0.132)) * (1 - 3.3/24) = ~460kHz\n  Eq.20: L_min = Vin(max) * ton(min) / IL(max)\n         = 45V * 180ns / 0.25A = 32.4uH  -> 47uH OK\n\nC_OUT = 10uF, 10V, X7R, 0805\n  Eq.22: Cout >= 100 * L * (Ipk/Vout)^2\n         = 100 * 47u * (0.132/3.3)^2 = 7.5uF  -> 10uF OK\n  Eq.21: dVout = Iout*4us/Cout + Vout/123\n         @12mA = 4.8mV + 26.8mV = ~32mV pk-pk\n\nC_IN = 1uF, 100V, X7R (rating >= 2x Vin(max))\n  Add 4.7uF electrolytic bulk if source > ~5cm away\n\nPIN CONFIG:\n  VOUT  -> output node (internal FB divider, Y version)\n  EN    -> VIN (always on)\n  SS    -> open (internal 900us soft start)\n  HYS   -> open\n  PGOOD -> optional: 100k pull-up to 3.3V ONLY (abs max 16V)\n           rises at 94% Vout (~3.1V), falls at 87% (~2.87V)\n  PAD   -> GND with thermal vias"
+	(text "LM5165Y-Q1  24V -> 3.3V  PFM MODE  (ref: TI SNVSAJ3C, Design 2)\nVin(nom)=24V  Vin(op)=24-28V  Vin(max)=32V (rail limit, TPS56A37 abs max)\nVout=3.3V (fixed, Y version)  Iout(target)=50mA  Iout(max)=60mA\n\nMODE: RT tied to GND -> PFM (light-load efficiency)\n\nR_ILIM = 56.2k (1%) -> Ipk = 120mA\n  PFM: Iout(max) = Ipk/2 = 60mA  (design target 50mA)\n\nL_F = 47uH, Isat >= 0.5A  (Coilcraft LPS4018-473MRC)\n  Eq.19: Fsw = (Vout/(L*Ipk)) * (1 - Vout/Vin)\n         Ipk = 120mA * 1.1 = 132mA (comparator delay margin)\n         Fsw @24V = (3.3/(47u*0.132)) * (1 - 3.3/24) = ~459kHz\n         Fsw @28V = (3.3/(47u*0.132)) * (1 - 3.3/28) = ~469kHz\n  Eq.20: L_min = Vin(max) * ton(min) / IL(max)\n         = 32V * 180ns / 0.25A = 23.0uH  -> 47uH OK\n         (still OK at 45V: 32.4uH)\n  Isat margin: 0.5A >> Ipk 132mA OK\n\nC_OUT = 22uF, 10V, X7R, 0805  (~11uF eff @3.3V DC bias)\n  Eq.22: Cout >= 100 * L * (Ipk/Vout)^2\n         = 100 * 47u * (0.132/3.3)^2 = 7.5uF  -> 11uF eff OK\n  Eq.21: dVout = Iout*4us/Cout + Vout/123\n         @12mA = 12m*4u/11u + 3.3/123 = 4.4mV + 26.8mV = ~31mV pk-pk\n\nC_IN = 1uF, 100V, X7R  (rating >= 2x Vin(max) = 64V OK)\n  Bulk: shared 100uF 50V electrolytic (C1) at 24V input connector\n  D1 SMBJ26A TVS footprint at connector: DNP\n    -> populate if hot-plug scope peak on VIN > ~30V\n\nPIN CONFIG:\n  VOUT   -> output node (internal FB divider, Y version)\n  EN     -> VIN (always on)\n  SS     -> open (internal 900us soft start)\n  HYS    -> open\n  PGOOD  -> optional: 100k pull-up to 3.3V ONLY (abs max 16V)\n            rises at 94% Vout (~3.1V), falls at 87% (~2.87V)\n  RT     -> GND (PFM mode)\n  ILIM   -> 56.2k to GND\n  PAD    -> GND with thermal vias"
 		(exclude_from_sim no)
 		(at 129.54 93.98 0)
 		(effects
 			(font
-				(size 1.27 1.27)
+				(size 1.016 1.016)
 			)
 			(justify left)
@@
 			)
 		)
-		(property "Value" "10u"
+		(property "Value" "22u"
 			(at 283.21 90.1699 0)
 			(show_name no)
@@
 			)
 		)
-		(property "Footprint" ""
+		(property "Footprint" "Library:IND_LPS4018-473MRC"
 			(at 267.97 83.82 0)
 			(hide yes)
@@
 			)
 		)
-		(property "Footprint" ""
+		(property "Footprint" "Connector_BarrelJack:BarrelJack_CUI_PJ-063AH_Horizontal"
 			(at 317.5 175.006 90)
 			(hide yes)
@@
 			)
 		)
-		(property "Footprint" ""
+		(property "Footprint" "Library:L_Wurth_WE-HCI-1890"
 			(at 232.41 160.02 0)
 			(hide yes)
@@
 			)
 		)
-		(property "Datasheet" ""
+		(property "Datasheet" "www.we-online.com/components/products/datasheet/7443556560.pdf"
 			(at 232.41 160.02 0)
 			(hide yes)

Commit message: Adding some DRC constraints. Must finish adding stackup and predefined sizes
Parts:
- removed BT1: 5V (Battery_Cell), Connector_BarrelJack:BarrelJack_CUI_PJ-063AH_Horizontal, symbol Device:Battery_Cell
